File: pcb/ece49022-interface/RP2350_60QFN_minimal.kicad_sch (KiCad schematic)
At the start: 43 parts, among them J1 USB_B_Micro, J2 Conn_02x18_Odd_Even, J3 Conn_02x18_Odd_Even, J4 SM03B-SRSS-TB, SW1 SW_Push, SW2 SW_Push, U1 RP2350_60QFN, U2 NCP1117-3.3_SOT223, U3 W25Q128JVS, Y1 ABM8-272-T3

Commit message: interface
Parts:
- removed C1, C5: 10u, Capacitor_SMD:C_0805_2012Metric, symbol Device:C
- removed J1: USB_B_Micro, Connector_USB:USB_Micro-B_Amphenol_10103594-0001LF_Horizontal, symbol Connector:USB_B_Micro
- removed J2, J3: Conn_02x18_Odd_Even, Connector_PinHeader_2.54mm:PinHeader_2x18_P2.54mm_Vertical, symbol Connector_Generic:Conn_02x18_Odd_Even
- removed U2: NCP1117-3.3_SOT223, Package_TO_SOT_SMD:SOT-223-3_TabPin2, symbol Regulator_Linear:NCP1117-3.3_SOT223
Connections:
- no-connect marks 1 -> 0
Other:
- note removed: "IOs"
- note removed: "Power"
