File: pcb/ece49022-interface/buzzerdriver.kicad_sch (KiCad schematic)
At the start: 0 parts

Commit message: Buzzer
Updated buzzer schematic
Parts:
- added Q1: C1815, symbol Simulation_SPICE:NPN
- added R2, R3: 1k, 5%, symbol Device:R_US
- added XTAL1: PS1240P02BT, XTAL_PS1240P02BT_TDK, symbol PS1240P02BT Buzzer:PS1240P02BT
Connections:
- new net: Q1.1 (C), R3.1, XTAL1.2
- new net: Q1.2 (B), R2.2
- new net +5V: R3.2, XTAL1.1
- new net Buzzer_PWM: R2.1
- new net GND: Q1.3 (E)

Commit message: Update
Parts:
- renumbered XTAL1 to Buzzer
Other:
- moved on the sheet: BuzzerA, Q1, R2, R3
