File: pcb/ece49022-interface/ece49022-interface.kicad_pcb (KiCad board)
At the start: 4 copper layers, 68.4 x 52.2 mm, 38 parts, among them J1 Conn_01x03_Pin, J2 Conn_01x05_Pin, J3 Conn_01x04_Pin, J4 Conn_01x04_Pin, J5 Conn_01x02_Pin, J6 Conn_01x02_Pin, Q1 KSC1815, U4 NCP1117-3.3_SOT223, U5 TPS54202DDCT

Commit message: update
Parts:
- moved J2 21.1 mm to (124.4, 85.4)
- moved C21 11.5 mm to (139.3, 115.9)
- moved C23 11.5 mm to (137.6, 114.7)
- moved C24 11.5 mm to (128.8, 101.1)
- moved C26 11.5 mm to (139.3, 109.6)
- moved C27 11.5 mm to (140.8, 100.6)
- moved C29 11.5 mm to (138.4, 106.0)
- moved C31 11.5 mm to (140.8, 106.0)
- moved L2 11.5 mm to (131.4, 109.8)
- moved R12 11.5 mm to (141.1, 114.8)
- moved R13 11.5 mm to (141.1, 116.8)
- moved R17 11.5 mm to (143.8, 107.5)
- moved R18 11.5 mm to (142.3, 113.4)
- moved U5 11.5 mm to (139.3, 112.0)
- moved C33 11.5 mm to (142.7, 107.5)
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Connections:
- A1 pad 11: unconnected-(A1-GPIO8-Pad11) -> /BC_Rx
- A1 pad 12: unconnected-(A1-GPIO9-Pad12) -> /BC_Tx
- A1 pad 16: /BC_Rx -> unconnected-(A1-GPIO12-Pad16)
- A1 pad 17: /BC_Tx -> unconnected-(A1-GPIO13-Pad17)
Routing:
- net /BC_Tx: track 24.4 -> 0.00 mm
- net /BC_Rx: track 24.4 -> 0.00 mm
- net Net-(A1-GPIO4): track 18.8 -> 17.1 mm
- net unconnected-(A1-GPIO13-Pad17): track 0.00 -> 1.09 mm
- net unconnected-(A1-GPIO12-Pad16): track 0.00 -> 0.91 mm
