File: pcb/ece49022-interface/ece49022-interface.kicad_pcb (KiCad board)
At the start: 4 copper layers, 68.4 x 52.2 mm, 38 parts, among them J1 Conn_01x03_Pin, J2 Conn_01x05_Pin, J3 Conn_01x04_Pin, J4 Conn_01x04_Pin, J5 Conn_01x02_Pin, J6 Conn_01x02_Pin, Q1 KSC1815, U4 NCP1117-3.3_SOT223, U5 TPS54202DDCT

Commit message: Initial PCB
Parts:
- removed C24, C27: 10u, Capacitor_SMD:C_0805_2012Metric
- removed U4: NCP1117-3.3_SOT223, Package_TO_SOT_SMD:SOT-223-3_TabPin2
- moved J6 26.4 mm to (140.0, 120.7), turned to 90 degrees
- moved J2 8.44 mm to (129.5, 92.1)
- moved J4 8.26 mm to (129.5, 80.5)
- moved R4 7.91 mm to (137.0, 83.6)
- moved R5 7.84 mm to (137.0, 84.7)
- moved R6 7.78 mm to (137.0, 85.8)
- moved Buzzer1 4.20 mm to (173.8, 113.2), turned to 0 degrees
- moved R18 2.74 mm to (144.9, 114.3)
- moved R13 2.40 mm to (143.5, 116.8)
- moved C33 2.30 mm to (144.9, 108.2)
- moved C26 2.01 mm to (141.0, 110.7)
- moved L2 1.97 mm to (132.8, 111.2)
- moved C21 1.91 mm to (140.9, 116.9), turned to 0 degrees
- moved J1 1.90 mm to (185.5, 92.6)
- moved J3 1.90 mm to (185.5, 106.9)
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Connections:
- A1 pad 36: unconnected-(A1-3V3-Pad36) -> +3V3
Routing:
- net /MAIN_MCU_I2C_SDA: track 0.00 -> 21.7 mm
- net /MAIN_MCU_I2C_SCL: track 0.00 -> 20.8 mm
- net Net-(U5-SW): track 11.1 -> 0.00 mm, vias 0 -> 4
- net Net-(A1-GPIO3): track 18.5 -> 10.8 mm
- net Net-(A1-GPIO4): track 17.1 -> 10.6 mm
- net Net-(A1-GPIO2): track 17.8 -> 11.4 mm
- net Net-(Q1-C): track 6.87 -> 13.1 mm, vias 0 -> 2
- net Net-(U5-EN): track 1.04 -> 6.29 mm, vias 0 -> 2
- net +5V: track 0.00 -> 3.49 mm, vias 0 -> 1
- net +12V: track 0.00 -> 2.63 mm
- net GND: track 0.00 -> 2.62 mm, vias 0 -> 18
- net /PWM_B: track 5.62 -> 7.87 mm
- net /FS_Rx: track 23.3 -> 21.2 mm
- net /GPIO28: track 21.9 -> 19.8 mm
- net /GPIO22: track 7.11 -> 5.08 mm
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- added copper zone on F.Cu, net +12V
- added copper zone on F.Cu, net +3V3
- added copper zone on B.Cu, net +5V
- added copper zone on F.Cu, net GND
- added copper zone on F.Cu, net Net-(U5-BOOT)
- added copper zone on B.Cu, net Net-(U5-SW)
- added copper zone on F.Cu, net Net-(U5-SW)
- removed copper zone on B.Cu, net +3V3
Other:
- board size 68.4 x 52.2 mm -> 61 x 52.2 mm

Commit message: done? i think
Parts:
- moved J1 58.6 mm to (129.7, 110.5), turned to 0 degrees
- moved J4 56.5 mm to (185.5, 88.4)
- moved R1 46.5 mm to (137.8, 116.8), turned to -90 degrees
- moved MOSFET1 44.2 mm to (136.9, 113.7), turned to 90 degrees
- moved D5 42.5 mm to (136.1, 110.4), turned to 0 degrees
- moved R6 42.0 mm to (178.1, 94.3), turned to 180 degrees
- moved R4 42.0 mm to (178.1, 92.1), turned to 180 degrees
- moved R5 42.0 mm to (178.1, 93.2), turned to 180 degrees
- moved J6 20.8 mm to (129.7, 102.6), turned to 180 degrees
- moved L2 16.8 mm to (138.7, 95.5), turned to 0 degrees
- moved C21 15.5 mm to (133.0, 103.6), turned to -90 degrees
- moved R13 14.9 mm to (133.1, 106.2), turned to 180 degrees
- moved C23 14.1 mm to (134.6, 102.0), turned to -90 degrees
- moved R12 12.9 mm to (134.6, 105.0), turned to -90 degrees
- moved J2 12.4 mm to (129.7, 79.8)
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Connections:
- A1 pad 11: /BC_Rx -> unconnected-(A1-GPIO8-Pad11)
- A1 pad 12: /BC_Tx -> unconnected-(A1-GPIO9-Pad12)
- A1 pad 17: unconnected-(A1-GPIO13-Pad17) -> /GPIO13
- A1 pad 31: unconnected-(A1-GPIO26_ADC0-Pad31) -> Net-(A1-GPIO26_ADC0)
- A1 pad 32: unconnected-(A1-GPIO27_ADC1-Pad32) -> Net-(A1-GPIO27_ADC1)
- A1 pad 34: /GPIO28 -> Net-(A1-GPIO28_ADC2)
- A1 pad 4: Net-(A1-GPIO2) -> unconnected-(A1-GPIO2-Pad4)
- A1 pad 5: Net-(A1-GPIO3) -> unconnected-(A1-GPIO3-Pad5)
- A1 pad 6: Net-(A1-GPIO4) -> /BC_Rx
- A1 pad 7: unconnected-(A1-GPIO5-Pad7) -> /BC_Tx
- J1 pad 3: /GPIO28 -> /GPIO13
- MOSFET1 pad 1: /GPIO28 -> /GPIO13
- R1 pad 1: /GPIO28 -> /GPIO13
- R4 pad 2: Net-(A1-GPIO2) -> Net-(A1-GPIO28_ADC2)
- R5 pad 2: Net-(A1-GPIO3) -> Net-(A1-GPIO27_ADC1)
- R6 pad 2: Net-(A1-GPIO4) -> Net-(A1-GPIO26_ADC0)
Routing:
- net /GPIO28: track 19.8 -> 0.00 mm
- net /LOCK_RTN: track 18.3 -> 2.43 mm, vias 2 -> 0
- net GND: track 2.62 -> 17.0 mm, vias 18 -> 19
- net /GPIO13: track 0.00 -> 11.9 mm
- net Net-(A1-GPIO28_ADC2): track 0.00 -> 11.8 mm
- net Net-(A1-GPIO26_ADC0): track 0.00 -> 11.4 mm
- net Net-(A1-GPIO2): track 11.4 -> 0.00 mm
- net Net-(A1-GPIO3): track 10.8 -> 0.00 mm
- net Net-(A1-GPIO4): track 10.6 -> 0.00 mm
- net Net-(A1-GPIO27_ADC1): track 0.00 -> 10.4 mm
- net +5V: track 3.49 -> 4.64 mm, vias 1 -> 5
- net /PWM_R: track 7.13 -> 7.78 mm
Other:
- board size 61 x 52.2 mm -> 60.2 x 52.2 mm

Commit message: oshkosh drc
Routing:
- net /BC_Tx: track 0.00 -> 19.2 mm
- net /BC_Rx: track 0.00 -> 19.1 mm
- net /GPIO13: track 11.9 -> 20.3 mm
- net /LOCK_RTN: track 2.43 -> 10.6 mm
- net GND: track 17.0 -> 20.9 mm, vias 19 -> 20
Changed lines of the file:
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@@
+	)
+	(segment
+		(start 148.02 116.82)
+		(end 144.28 116.82)
+		(width 0.2)
+		(layer "F.Cu")
+		(net 5)
 	)
 	(segment
@@
 	)
 	(segment
+		(start 144.28 116.82)
+		(end 144.2 116.9)
+		(width 0.2)
+		(layer "F.Cu")
+		(net 5)
+	)
+	(segment
 		(start 148.02 78.72)
 		(end 144.52 78.72)
@@
 	)
 	(via
-		(at 134.8 112.9)
+		(at 134.8 113.7)
 		(size 0.6)
 		(drill 0.3)
@@
 	)
 	(via
-		(at 134.8 113.7)
+		(at 134.8 114.5)
 		(size 0.6)
 		(drill 0.3)
@@
 	)
 	(via
+		(at 144.2 116.9)
+		(size 0.6)
+		(drill 0.3)
+		(layers "F.Cu" "B.Cu")
+		(free yes)
+		(net 5)
+	)
+	(via
 		(at 138.7 100.7)
 		(size 0.6)
@@
 	)
 	(via
-		(at 134.8 114.5)
+		(at 134.8 115.3)
 		(size 0.6)
 		(drill 0.3)
@@
 	)
 	(segment
+		(start 131.34 88.3)
+		(end 147.44 88.3)
+		(width 0.2)
+		(layer "F.Cu")
+		(net 10)
+	)
+	(segment
+		(start 129.7 89.94)
+		(end 131.34 88.3)
+		(width 0.2)
+		(layer "F.Cu")
+		(net 10)
+	)
+	(segment
+		(start 147.44 88.3)
+		(end 148.02 88.88)
+		(width 0.2)
+		(layer "F.Cu")
+		(net 10)
+	)
+	(segment
 		(start 168.44 120.4)
 		(end 177.06 120.4)
@@
 		(layer "F.Cu")
 		(net 17)
+	)
+	(segment
+		(start 148.02 86.34)
+		(end 145.96 86.34)
+		(width 0.2)
+		(layer "F.Cu")
+		(net 18)
+	)
+	(segment
+		(start 130 87.7)
+		(end 129.7 87.4)
+		(width 0.2)
+		(layer "F.Cu")
+		(net 18)
+	)
+	(segment
+		(start 144.7 87.7)
+		(end 145.96 86.44)
+		(width 0.2)
+		(layer "F.Cu")
+		(net 18)
+	)
+	(segment
+		(start 145.96 86.44)
+		(end 145.96 86.34)
+		(width 0.2)
+		(layer "F.Cu")
+		(net 18)
+	)
+	(segment
+		(start 144.7 87.7)
+		(end 130 87.7)
+		(width 0.2)
+		(layer "F.Cu")
+		(net 18)
 	)
 	(segment
@@
 	)
 	(segment
+		(start 129.7 113)
+		(end 129.8 113)
+		(width 0.2)
+		(layer "F.Cu")
+		(net 29)
+	)
+	(segment
 		(start 137.713099 112.566251)
 		(end 137.713099 110.391251)
@@
 	)
 	(segment
+		(start 129.8 113)
+		(end 130.023748 112.776252)
+		(width 0.2)
+		(layer "F.Cu")
+		(net 29)
+	)
+	(segment
 		(start 137.816899 112.776252)
 		(end 137.816899 112.670051)
@@
 	)
 	(segment
+		(start 130.023748 112.776252)
+		(end 137.816899 112.776252)
+		(width 0.2)
+		(layer "F.Cu")
+		(net 29)
+	)
+	(segment
 		(start 175.435 100.2)
 		(end 175.9 99.735)
@@
 	)
 	(segment
+		(start 131.423149 116.176851)
+		(end 137.8 116.176851)
+		(width 0.2)
+		(layer "F.Cu")
+		(net 47)
+	)
+	(segment
 		(start 137.816899 114.60625)
 		(end 147.69375 114.60625)
@@
 	)
 	(segment
+		(start 129.7 115.54)
+		(end 130.74 115.54)
+		(width 0.2)
+		(layer "F.Cu")
+		(net 47)
+	)
+	(segment
 		(start 137.8 116.176851)
 		(end 137.8 114.623149)
@@
 	)
 	(segment
+		(start 130.74 115.54)
+		(end 131.4 116.2)
+		(width 0.2)
+		(layer "F.Cu")
+		(net 47)
+	)
+	(segment
 		(start 137.8219 114.611251)
 		(end 137.816899 114.60625)
+		(width 0.2)
+		(layer "F.Cu")
+		(net 47)
+	)
+	(segment
+		(start 131.4 116.2)
+		(end 131.423149 116.176851)
 		(width 0.2)
 		(layer "F.Cu")
@@
 		(polygon
 			(pts
-				(xy 134.4 112.5) (xy 136.1 112.5) (xy 136.1 114.9) (xy 134.4 114.9)
+				(xy 134.4 113.3) (xy 136.1 113.3) (xy 136.1 115.7) (xy 134.4 115.7)
 			)
 		)

Commit message: need to finish power
Parts:
- J5: value Conn_01x02_Pin -> Conn_01x08_Pin; footprint Connector_PinHeader_2.54mm:PinHeader_1x02_P2.54mm_Vertical -> Connector_PinHeader_2.54mm:PinHeader_1x08_P2.54mm_Vertical
- moved J1 58.6 mm to (185.6, 92.8), turned to 180 degrees
- moved J4 57.4 mm to (129.8, 74.7)
- moved J6 55.9 mm to (185.6, 100.6), turned to 0 degrees
- moved J5 55.7 mm to (129.9, 100.1), turned to 0 degrees
- moved R13 49.9 mm to (182.2, 97.0), turned to 0 degrees
- moved R1 49.9 mm to (177.4, 86.5), turned to 90 degrees
- moved C21 49.4 mm to (182.2, 99.6), turned to 90 degrees
- moved MOSFET1 48.0 mm to (178.3, 89.6), turned to -90 degrees
- moved R12 46.5 mm to (180.7, 98.2), turned to 90 degrees
- moved D5 46.4 mm to (179.1, 92.9), turned to 180 degrees
- moved C23 46.1 mm to (180.7, 101.2), turned to 90 degrees
- moved R18 45.6 mm to (179.7, 95.6), turned to 0 degrees
- moved R4 42.8 mm to (137.0, 80.1), turned to 0 degrees
- moved R6 42.8 mm to (137.0, 82.3), turned to 0 degrees
- moved R5 42.8 mm to (137.0, 81.2), turned to 0 degrees
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Connections:
- A1 pad 14: unconnected-(A1-GPIO10-Pad14) -> /GPIO10
- A1 pad 16: unconnected-(A1-GPIO12-Pad16) -> /MAIN_MCU_I2C_SDA
- A1 pad 17: /GPIO13 -> /MAIN_MCU_I2C_SCL
- A1 pad 2: unconnected-(A1-GPIO1-Pad2) -> Net-(A1-GPIO1)
- A1 pad 26: /MAIN_MCU_I2C_SDA -> unconnected-(A1-GPIO20-Pad26)
- A1 pad 27: /MAIN_MCU_I2C_SCL -> unconnected-(A1-GPIO21-Pad27)
- A1 pad 29: /GPIO22 -> unconnected-(A1-GPIO22-Pad29)
- A1 pad 31: Net-(A1-GPIO26_ADC0) -> unconnected-(A1-GPIO26_ADC0-Pad31)
- A1 pad 32: Net-(A1-GPIO27_ADC1) -> unconnected-(A1-GPIO27_ADC1-Pad32)
- A1 pad 34: Net-(A1-GPIO28_ADC2) -> /GPIO28
- A1 pad 4: unconnected-(A1-GPIO2-Pad4) -> Net-(A1-GPIO2)
- A1 pad 5: unconnected-(A1-GPIO3-Pad5) -> Net-(A1-GPIO3)
- J1 pad 3: /GPIO13 -> /GPIO28
- J2 pad 4: /BC_Rx -> /BC_Tx
- J2 pad 5: /BC_Tx -> /BC_Rx
- J5 pad 2: /MAIN_MCU_I2C_SCL -> /MAIN_MCU_I2C_SDA
- MOSFET1 pad 1: /GPIO13 -> /GPIO28
- R1 pad 1: /GPIO13 -> /GPIO28
- R2 pad 1: /GPIO22 -> /GPIO10
- R4 pad 2: Net-(A1-GPIO28_ADC2) -> Net-(A1-GPIO1)
- R5 pad 2: Net-(A1-GPIO27_ADC1) -> Net-(A1-GPIO2)
- R6 pad 2: Net-(A1-GPIO26_ADC0) -> Net-(A1-GPIO3)
Routing:
- net /GPIO13: track 20.3 -> 0.00 mm
- net /GPIO28: track 0.00 -> 20.1 mm
- net /MAIN_MCU_I2C_SDA: track 21.7 -> 35.9 mm
- net Net-(A1-GPIO1): track 0.00 -> 12.0 mm
- net Net-(A1-GPIO28_ADC2): track 11.8 -> 0.00 mm
- net /MAIN_MCU_I2C_SCL: track 20.8 -> 32.5 mm
- net Net-(A1-GPIO26_ADC0): track 11.4 -> 0.00 mm
- net Net-(A1-GPIO3): track 0.00 -> 11.0 mm
- net Net-(A1-GPIO2): track 0.00 -> 10.4 mm
- net Net-(A1-GPIO27_ADC1): track 10.4 -> 0.00 mm
- net /GPIO10: track 0.00 -> 5.54 mm
- net /GPIO22: track 5.08 -> 0.00 mm
- net Net-(Q1-C): track 13.1 -> 10.7 mm, vias 2 -> 0
- net GND: track 20.9 -> 22.9 mm, vias 20 -> 21
- net /PWM_B: track 8.01 -> 6.62 mm

Commit message: need to figure out lock circuit
Parts:
- J1: value Conn_01x03_Pin -> Conn_01x04_Pin; footprint Connector_PinHeader_2.54mm:PinHeader_1x03_P2.54mm_Vertical -> Connector_PinHeader_2.54mm:PinHeader_1x04_P2.54mm_Vertical
- moved J1 7.57 mm to (185.6, 85.2), turned to 0 degrees
Connections:
- A1 pad 32: unconnected-(A1-GPIO27_ADC1-Pad32) -> /GPIO27
- J1 pad 1: +12V -> GND
- J1 pad 2: /LOCK_RTN -> /GPIO27
- J1 pad 3: /GPIO28 -> /LOCK_RTN
- MOSFET1 pad 1: /GPIO28 -> /GPIO27
- R1 pad 1: /GPIO28 -> /GPIO27
Routing:
- net /GPIO27: track 0.00 -> 22.8 mm
- net /GPIO28: track 20.1 -> 0.00 mm

Commit message: lock state
Parts:
- added R7: 10K, 1%, Resistor_SMD:R_0402_1005Metric_Pad0.72x0.64mm_HandSolder, F.Cu at (173.0, 84.7)
- added R8: 10K, 1%, Resistor_SMD:R_0402_1005Metric_Pad0.72x0.64mm_HandSolder, F.Cu at (173.0, 85.8)
- moved R1 3.31 mm to (175.0, 88.7), turned to 180 degrees
Connections:
- J1 pad 1: GND -> /LOCK_RTN
- J1 pad 2: /GPIO27 -> /LOCK_STATUS
- J1 pad 3: /LOCK_RTN -> +5V
Routing:
- net /GPIO27: track 22.8 -> 0.00 mm
- net /LOCK_RTN: track 10.6 -> 0.00 mm

Commit message: update
Parts:
- removed C21: 22uF, Capacitor_SMD:C_0805_2012Metric_Pad1.18x1.45mm_HandSolder
- removed C23, C26: 0.1uF, Capacitor_SMD:C_0402_1005Metric
- removed C29, C31: 22uF,25V, Capacitor_SMD:C_0805_2012Metric_Pad1.18x1.45mm_HandSolder
- removed C33: 75pF, Capacitor_SMD:C_0402_1005Metric
- removed R16: 49.9, 1%, Capacitor_SMD:C_0402_1005Metric
- removed R17: 100k, 1%, Capacitor_SMD:C_0402_1005Metric
- removed R18: 13.3k, 1%, Capacitor_SMD:C_0402_1005Metric
- removed U5: TPS54202DDCT, 49022_Footprints:TPS54202
- added C10: 22uF,25V, Capacitor_SMD:C_0805_2012Metric_Pad1.18x1.45mm_HandSolder, F.Cu at (172.4, 101.3)
- added C11: 22uF,25V, Capacitor_SMD:C_0805_2012Metric_Pad1.18x1.45mm_HandSolder, F.Cu at (172.4, 99.2)
- added C12: 75pF, Capacitor_SMD:C_0402_1005Metric, F.Cu at (173.5, 96.5)
- added C7: 22uF, Capacitor_SMD:C_1206_3216Metric, F.Cu at (181.9, 99.4)
- added C8: 0.1uF, Capacitor_SMD:C_0402_1005Metric, F.Cu at (179.7, 97.1)
- added C9: 0.1uF, Capacitor_SMD:C_0402_1005Metric, F.Cu at (177.9, 101.8)
- added R10: 105k, Capacitor_SMD:C_0402_1005Metric, F.Cu at (175.7, 100.6)
- added R14: 13.3k, 1%, Capacitor_SMD:C_0402_1005Metric, F.Cu at (177.7, 97.1)
- added R9: 510K, Capacitor_SMD:C_0402_1005Metric, F.Cu at (175.7, 98.5)
- added U2: TPS54202DDCT, 49022_Footprints:TPS54202, F.Cu at (178.5, 99.4)
- R12: value 0 -> 49.9, 1%
- R13: value 0 -> 100k, 1%
- moved R12 9.15 mm to (171.5, 97.6), turned to 0 degrees
- moved R13 8.67 mm to (173.5, 97.6)
- moved J6 3.88 mm to (185.6, 96.7)
- moved R7 3.71 mm to (173.9, 88.3), turned to -90 degrees
- moved R8 2.52 mm to (172.7, 88.3), turned to 90 degrees
- moved R1 0.99 mm to (175.7, 89.4), turned to -90 degrees
- moved Buzzer1 0.70 mm to (136.0, 95.7)
- moved L2 0.21 mm to (176.4, 107.8)
- moved J3 0.11 mm to (185.6, 107.8)
Connections:
- J1 pad 1: /LOCK_RTN -> /LOCK_STATUS
- J1 pad 2: /LOCK_STATUS -> /LOCK_RTN
- R12 pad 1: +12V -> +5V
- R13 pad 2: GND -> /Power/FB
Routing:
- net /GPIO27: track 0.00 -> 12.9 mm
- net +12V: track 2.63 -> 15.4 mm
- net /LOCK_STATUS: track 0.00 -> 12.7 mm
- net /LOCK_RTN: track 0.00 -> 12.5 mm
- net /GPIO28: track 0.00 -> 7.13 mm
- net Net-(C12-Pad1): track 6.29 -> 2.14 mm, vias 2 -> 0
- net /Power/FB: track 9.35 -> 5.89 mm, vias 0 -> 2
- net GND: track 22.9 -> 25.9 mm, vias 21 -> 32
- net Net-(U2-EN): track 0.00 -> 2.73 mm
- net Net-(C33-Pad1): track 2.57 -> 0.00 mm
- net +5V: track 4.80 -> 3.03 mm, vias 5 -> 4
- net /MAIN_MCU_I2C_SCL: track 32.5 -> 33.8 mm
- net /MAIN_MCU_I2C_SDA: track 35.9 -> 36.6 mm
- net Net-(U2-SW): vias 4 -> 10
- added copper zone on F.Cu, net Net-(U2-BOOT)
- removed copper zone on F.Cu, net Net-(U5-BOOT)

Commit message: +5V
Routing:
- net +5V: track 3.03 -> 30.2 mm, vias 4 -> 5
- net +12V: track 15.4 -> 20.3 mm
- net GND: track 25.9 -> 27.4 mm, vias 32 -> 34
Changed lines of the file:
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@@
+	)
+	(segment
+		(start 178.7 96.45)
+		(end 178.7 97.117378)
+		(width 0.5)
+		(layer "F.Cu")
+		(net 3)
 	)
 	(segment
@@
 	)
 	(segment
+		(start 178.7 97.117378)
+		(end 179.2 97.117378)
+		(width 0.5)
+		(layer "F.Cu")
+		(net 3)
+	)
+	(segment
 		(start 145.12 78.72)
 		(end 145.1 78.7)
@@
 	(segment
 		(start 178.2 97.117378)
-		(end 179.2 97.117378)
+		(end 178.7 97.117378)
 		(width 0.5)
 		(layer "F.Cu")
@@
 	)
 	(segment
+		(start 175.7 101.077378)
+		(end 175.7 101.9)
+		(width 0.2)
+		(layer "F.Cu")
+		(net 3)
+	)
+	(segment
 		(start 148.02 91.42)
 		(end 145.08 91.42)
@@
 	)
 	(via
+		(at 178.7 96.45)
+		(size 0.6)
+		(drill 0.3)
+		(layers "F.Cu" "B.Cu")
+		(free yes)
+		(net 3)
+	)
+	(via
 		(at 169.3 104.1)
 		(size 0.6)
@@
 	(via
 		(at 144.1 116.9)
+		(size 0.6)
+		(drill 0.3)
+		(layers "F.Cu" "B.Cu")
+		(free yes)
+		(net 3)
+	)
+	(via
+		(at 175.7 101.9)
 		(size 0.6)
 		(drill 0.3)
@@
 	)
 	(segment
+		(start 171.325 99.217378)
+		(end 171.325 101.317378)
+		(width 0.5)
+		(layer "F.Cu")
+		(net 16)
+	)
+	(segment
 		(start 137.7025 102.8225)
 		(end 136.4225 102.8225)
@@
 	)
 	(segment
+		(start 171.04 97.617378)
+		(end 171.04 96.21)
+		(width 0.5)
+		(layer "F.Cu")
+		(net 16)
+	)
+	(segment
+		(start 171.325 101.317378)
+		(end 171.325 107.484878)
+		(width 0.5)
+		(layer "F.Cu")
+		(net 16)
+	)
+	(segment
 		(start 136.4225 102.8225)
 		(end 136.4 102.8)
@@
 		(net 16)
 	)
+	(segment
+		(start 174.15 93.1)
+		(end 175.8 93.1)
+		(width 0.5)
+		(layer "F.Cu")
+		(net 16)
+	)
+	(segment
+		(start 171.325 107.484878)
+		(end 171.6575 107.817378)
+		(width 0.5)
+		(layer "F.Cu")
+		(net 16)
+	)
+	(segment
+		(start 171.04 96.21)
+		(end 174.15 93.1)
+		(width 0.5)
+		(layer "F.Cu")
+		(net 16)
+	)
 	(via
 		(at 179.6 77.5)
@@
 	)
 	(via
+		(at 175.8 93.1)
+		(size 0.6)
+		(drill 0.3)
+		(layers "F.Cu" "B.Cu")
+		(net 16)
+	)
+	(via
 		(at 136.4 102.8)
 		(size 0.6)
@@
 		(layers "F.Cu" "B.Cu")
 		(free yes)
+		(net 16)
+	)
+	(segment
+		(start 181.7 93.1)
+		(end 183.4 91.4)
+		(width 0.5)
+		(layer "B.Cu")
+		(net 16)
+	)
+	(segment
+		(start 184.5 91.4)
+		(end 183.4 91.4)
+		(width 0.5)
+		(layer "B.Cu")
+		(net 16)
+	)
+	(segment
+		(start 175.8 93.1)
+		(end 181.7 93.1)
+		(width 0.5)
+		(layer "B.Cu")
+		(net 16)
+	)
+	(segment
+		(start 185.6 90.3)
+		(end 184.5 91.4)
+		(width 0.5)
+		(layer "B.Cu")
 		(net 16)
 	)
@@
 		(start 182.475 96.725)
 		(end 185.6 96.725)
+		(width 0.5)
+		(layer "F.Cu")
+		(net 18)
+	)
+	(segment
+		(start 180.711901 92.853749)
+		(end 185.586251 92.853749)
 		(width 0.5)
 		(layer "F.Cu")
@@
 	)
 	(segment
-		(start 185.6 96.725)
-		(end 185.6 92.84)
+		(start 185.6 92.84)
+		(end 185.6 96.725)
 		(width 0.5)
 		(layer "F.Cu")
@@
 		(end 181.9 97.3)
 		(width 0.5)
+		(layer "F.Cu")
+		(net 18)
+	)
+	(segment
+		(start 185.586251 92.853749)
+		(end 185.6 92.84)
+		(width 0.2)
 		(layer "F.Cu")
 		(net 18)
@@
 			(pts
 				(xy 181.1 90.7) (xy 179.4 90.7) (xy 179.4 88.3) (xy 181.1 88.3)
-			)
-		)
-	)
-	(zone
-		(net 16)
-		(net_name "+5V")
-		(layer "F.Cu")
-		(hatch edge 0.5)
-		(priority 4)
-		(connect_pads
-			(clearance 0.15)
-		)
-		(min_thickness 0.25)
-		(filled_areas_thickness no)
-		(fill yes
-			(thermal_gap 0.5)
-			(thermal_bridge_width 0.5)
-		)
-		(polygon
-			(pts
-				(xy 172 98.417378) (xy 170.5 98.417378) (xy 170.55 109.767378) (xy 172.8 109.767378) (xy 172.8 105.717378)
-				(xy 172 105.717378)
 			)
 		)
@@
 		(polygon
 			(pts
-				(xy 179.8812 100.722178) (xy 179.8812 102.495378) (xy 183.8928 102.495378) (xy 183.8928 98.742578)
+				(xy 179.8812 100.872178) (xy 179.8812 102.495378) (xy 183.8928 102.495378) (xy 183.8928 98.742578)
 				(xy 182.2196 98.742578) (xy 182.2196 100.317378) (xy 180.44 100.317378) (xy 180.44 99.963378) (xy 178.67 99.963378)
-				(xy 178.67 100.722178)
+				(xy 178.67 100.872178)
 			)
 		)
