File: pcb/ece49022-shelf/_autosave-rp2350A.kicad_sch (KiCad schematic)
At the start: 33 parts, among them J1 USB_B_Micro, J4 SM03B-SRSS-TB, SW1 SW_Push, SW2 SW_Push, U3 W25Q128JVS, U5 RP2350_60QFN, Y1 ABM8-272-T3

Commit message: Started Layout
Connections:
- net FLASH_SS renamed QSPI_SS
Changed lines of the file:
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@@
 	(wire
 		(pts
-			(xy 24.13 123.19) (xy 58.42 123.19)
+			(xy 36.83 123.19) (xy 58.42 123.19)
 		)
 		(stroke
@@
 	)
 	(label "QSPI_SS"
-		(at 24.13 123.19 0)
+		(at 36.83 123.19 0)
 		(effects
 			(font
@@
 		)
 	)
-	(label "FLASH_SS"
-		(at 45.72 123.19 0)
-		(effects
-			(font
-				(size 1.27 1.27)
-			)
-			(justify left bottom)
-		)
-	)
