File: pcb/ece49022-shelf/_autosave-ece49022-shelf.kicad_sch (KiCad schematic)
At the start: 5 parts, among them J2 Conn_01x16_Pin, J3 Conn_01x04_Pin, J6 Conn_01x02_Pin, J7 Conn_01x02_Pin

Commit message: working n board
Parts:
- R11: footprint (none) -> Resistor_SMD:R_0805_2012Metric_Pad1.20x1.40mm_HandSolder
Changed lines of the file:
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@@
 			)
 		)
-		(property "Footprint" ""
+		(property "Footprint" "Resistor_SMD:R_0805_2012Metric_Pad1.20x1.40mm_HandSolder"
 			(at 179.07 105.41 0)
 			(effects
