File: pcb/ece49022-shelf/_autosave-NAU7802.kicad_sch (KiCad schematic)
At the start: 12 parts, among them IC1 NAU7802

Commit message: stuff
Parts:
- C1: footprint 49022_Footprints:C_0402_1005Metric_small_pads -> Capacitor_SMD:C_0402_1005Metric_Pad0.74x0.62mm_HandSolder
- C32, C5: footprint Capacitor_SMD:C_0402_1005Metric -> Capacitor_SMD:C_0402_1005Metric_Pad0.74x0.62mm_HandSolder
Changed lines of the file:
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@@
 			)
 		)
-		(property "Footprint" "Capacitor_SMD:C_0402_1005Metric"
+		(property "Footprint" "Capacitor_SMD:C_0402_1005Metric_Pad0.74x0.62mm_HandSolder"
 			(at 129.54 90.17 0)
 			(effects
@@
 			)
 		)
-		(property "Footprint" "49022_Footprints:C_0402_1005Metric_small_pads"
+		(property "Footprint" "Capacitor_SMD:C_0402_1005Metric_Pad0.74x0.62mm_HandSolder"
 			(at 165.1 113.03 0)
 			(effects
@@
 			)
 		)
-		(property "Footprint" "Capacitor_SMD:C_0402_1005Metric"
+		(property "Footprint" "Capacitor_SMD:C_0402_1005Metric_Pad0.74x0.62mm_HandSolder"
 			(at 147.32 86.36 0)
 			(effects
