File: pcb/ece49022-shelf/rp2350A.kicad_sch (KiCad schematic)
At the start: 32 parts, among them J1 USB_B_Micro, J4 Conn_01x03_Pin, SW1 SW_Push, SW2 SW_Push, U3 W25Q128JVS, U5 RP2350_60QFN, Y1 ABM8-272-T3

Commit message: layout chanes
Connections:
- net USB_DN: now reaches R19.2, U5.51 (USB_DM)
- net USB_DP: now reaches R18.2, U5.52 (USB_DP)
Changed lines of the file:
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@@
+		)
+	)
+	(label "USB_DP"
+		(at 231.14 92.71 0)
+		(effects
+			(font
+				(size 1.27 1.27)
+			)
+			(justify left bottom)
 		)
 	)
@@
 		)
 	)
+	(label "USB_DN"
+		(at 231.14 95.25 0)
+		(effects
+			(font
+				(size 1.27 1.27)
+			)
+			(justify left bottom)
+		)
+	)
