File: pcb/ece49022-shelf/power.kicad_sch (KiCad schematic)
At the start: 19 parts, among them U2 TPS54202DDCT, U4 NCP1117-3.3_SOT223

Commit message: fixed some stuff in interface and changed trace width for 50 ohm in shelf pcb
Parts:
- added D3, D4: LED, Resistor_SMD:R_0603_1608Metric, symbol Device:LED
- added R21, R22: 100, Resistor_SMD:R_0603_1608Metric, symbol Device:R_Small_US
Connections:
- net 5V_SREG: now also R21.1
- net 5V_USB: now also R22.1
- net GND: now also D3.1 (K), D4.1 (K)
- new net: D4.2 (A), R22.2
- new net: D3.2 (A), R21.2
Other:
- moved on the sheet: JP1
